File: accelerometer.sch (KiCad schematic (older format))
At the start: 7 parts, among them IC5 MMA7455

Commit message: pcb: refresh footprints, accelerometer deleted
Parts:
- C14, C16: footprint ~ -> Capacitors_Tantalum_SMD:TantalC_SizeB_EIA-3528_HandSoldering
- C15, C17: footprint ~ -> Capacitors_SMD:C_0805_HandSoldering
- IC5, R11, R12: footprint ~ -> (none)
Changed lines of the file:
@@
 F 0 "IC5" H 5850 4900 60  0000 C CNN
 F 1 "MMA7455" H 5850 4000 60  0000 C CNN
-F 2 "~" H 5850 4450 60  0000 C CNN
+F 2 "" H 5850 4450 60  0000 C CNN
 F 3 "~" H 5850 4450 60  0000 C CNN
 	1    5850 4450
@@
 F 0 "R11" V 6830 5200 40  0000 C CNN
 F 1 "4.7K" V 6757 5201 40  0000 C CNN
-F 2 "~" V 6680 5200 30  0000 C CNN
+F 2 "" V 6680 5200 30  0000 C CNN
 F 3 "~" H 6750 5200 30  0000 C CNN
 	1    6750 5200
@@
 F 0 "R12" V 7130 5200 40  0000 C CNN
 F 1 "4.7K" V 7057 5201 40  0000 C CNN
-F 2 "~" V 6980 5200 30  0000 C CNN
+F 2 "" V 6980 5200 30  0000 C CNN
 F 3 "~" H 7050 5200 30  0000 C CNN
 	1    7050 5200
@@
 F 0 "C15" H 5600 3050 40  0000 L CNN
 F 1 "0.1uF" H 5606 2865 40  0000 L CNN
-F 2 "~" H 5638 2800 30  0000 C CNN
+F 2 "Capacitors_SMD:C_0805_HandSoldering" H 5638 2800 30  0000 C CNN
 F 3 "~" H 5600 2950 60  0000 C CNN
 	1    5600 2950
@@
 F 0 "C17" H 6400 3050 40  0000 L CNN
 F 1 "0.1uF" H 6406 2865 40  0000 L CNN
-F 2 "~" H 6438 2800 30  0000 C CNN
+F 2 "Capacitors_SMD:C_0805_HandSoldering" H 6438 2800 30  0000 C CNN
 F 3 "~" H 6400 2950 60  0000 C CNN
 	1    6400 2950
@@
 F 0 "C16" H 6050 3050 50  0000 L CNN
 F 1 "10uF" H 6050 2850 50  0000 L CNN
-F 2 "~" H 6000 2950 60  0000 C CNN
+F 2 "Capacitors_Tantalum_SMD:TantalC_SizeB_EIA-3528_HandSoldering" H 6000 2950 60  0000 C CNN
 F 3 "~" H 6000 2950 60  0000 C CNN
 	1    6000 2950
@@
 F 0 "C14" H 5250 3050 50  0000 L CNN
 F 1 "10uF" H 5250 2850 50  0000 L CNN
-F 2 "~" H 5200 2950 60  0000 C CNN
+F 2 "Capacitors_Tantalum_SMD:TantalC_SizeB_EIA-3528_HandSoldering" H 5200 2950 60  0000 C CNN
 F 3 "~" H 5200 2950 60  0000 C CNN
 	1    5200 2950
