File: dc-motors_drivers.sch (KiCad schematic (older format))
At the start: 24 parts, among them IC3 L293DD, IC4 L293DD, P6 CONN_2, P7 CONN_2, P8 CONN_2, P9 CONN_2, U1 74HC595

Commit message: pcb: refresh footprints, accelerometer deleted
Parts:
- removed C10, C11, C12, C5, C6, C7, C8, C9: 1uF, ~, symbol C
- removed C13: 0.1uF, ~, symbol C
- added C10, C11, C12, C5, C6, C7, C8, C9: 1uF, Capacitors_SMD:C_0805_HandSoldering, symbol C_Small
- added C13: 0.1uF, Capacitors_SMD:C_0805_HandSoldering, symbol C_Small
- IC3, IC4: footprint ~ -> Housings_SOIC:SOIC-20_7.5x12.8mm_Pitch1.27mm
- P10: renamed from P9; footprint ~ -> Pin_Headers:Pin_Header_Angled_1x02
- P7: renamed from P6; footprint ~ -> Pin_Headers:Pin_Header_Angled_1x02
- P8: renamed from P7; footprint ~ -> Pin_Headers:Pin_Header_Angled_1x02
- P9: renamed from P8; footprint ~ -> Pin_Headers:Pin_Header_Angled_1x02
- R10, R3, R4, R5, R6, R7, R8, R9: footprint ~ -> Resistors_SMD:R_0805_HandSoldering
- U1: footprint ~ -> SMD_Packages:SO-16-N

Commit message: pcb: mma7455l replaced by mpu6050
Parts:
- renumbered C12 to C10, C13 to C11, C5 to C3, C6 to C4, C7 to C5, C8 to C6, C9 to C7, C10 to C8, C11 to C9, IC3 to IC2, IC4 to IC3, P7 to P6, P8 to P7, P9 to P8, P10 to P9
Connections:
- wire segments 150 -> 149

Commit message: pcb: ADC PCF85911 batery control added
Parts:
- removed P6, P7, P8, P9: CONN_2, Pin_Headers:Pin_Header_Angled_1x02, symbol CONN_2
- added P6, P7, P8, P9: CONN_01X02, Pin_Headers:Pin_Header_Angled_1x02, symbol CONN_01X02
- renumbered R6 to R10, R7 to R11, R8 to R12, R9 to R13, R10 to R14, R3 to R7, R4 to R8, R5 to R9, U1 to U2
