File: dc-motors_drivers.sch (KiCad schematic (older format))
At the start: 8 parts, among them J5 WHL_LF, J6 WHL_LB, J7 WHL_RF, J8 WHL_RB, U4 74HC595, U5 L293DD, U6 L293DD

Commit message: packages of PCB components was assigned
Parts:
- C17: value C -> 1uF; footprint (none) -> Capacitor_SMD:C_0805_2012Metric_Pad1.18x1.45mm_HandSolder
- J5, J6, J7, J8: footprint (none) -> Connector_JST:JST_PH_S2B-PH-K_1x02_P2.00mm_Horizontal
Changed lines of the file:
@@
 P 2350 3850
 F 0 "C17" H 2465 3896 50  0000 L CNN
-F 1 "C" H 2465 3805 50  0000 L CNN
-F 2 "" H 2388 3700 50  0001 C CNN
+F 1 "1uF" H 2465 3805 50  0000 L CNN
+F 2 "Capacitor_SMD:C_0805_2012Metric_Pad1.18x1.45mm_HandSolder" H 2388 3700 50  0001 C CNN
 F 3 "~" H 2350 3850 50  0001 C CNN
 	1    2350 3850
@@
 F 0 "J5" H 6730 2692 50  0000 L CNN
 F 1 "WHL_LF" H 6730 2601 50  0000 L CNN
-F 2 "" H 6650 2700 50  0001 C CNN
+F 2 "Connector_JST:JST_PH_S2B-PH-K_1x02_P2.00mm_Horizontal" H 6650 2700 50  0001 C CNN
 F 3 "~" H 6650 2700 50  0001 C CNN
 	1    6650 2700
@@
 F 0 "J7" H 8880 2692 50  0000 L CNN
 F 1 "WHL_RF" H 8880 2601 50  0000 L CNN
-F 2 "" H 8800 2700 50  0001 C CNN
+F 2 "Connector_JST:JST_PH_S2B-PH-K_1x02_P2.00mm_Horizontal" H 8800 2700 50  0001 C CNN
 F 3 "~" H 8800 2700 50  0001 C CNN
 	1    8800 2700
@@
 F 0 "J6" H 6730 4542 50  0000 L CNN
 F 1 "WHL_LB" H 6730 4451 50  0000 L CNN
-F 2 "" H 6650 4550 50  0001 C CNN
+F 2 "Connector_JST:JST_PH_S2B-PH-K_1x02_P2.00mm_Horizontal" H 6650 4550 50  0001 C CNN
 F 3 "~" H 6650 4550 50  0001 C CNN
 	1    6650 4550
@@
 F 0 "J8" H 8880 4542 50  0000 L CNN
 F 1 "WHL_RB" H 8880 4451 50  0000 L CNN
-F 2 "" H 8800 4550 50  0001 C CNN
+F 2 "Connector_JST:JST_PH_S2B-PH-K_1x02_P2.00mm_Horizontal" H 8800 4550 50  0001 C CNN
 F 3 "~" H 8800 4550 50  0001 C CNN
 	1    8800 4550

Commit message: preliminary PCB components placement
Parts:
- U4: footprint (none) -> Package_SO:SOP-16_4.4x10.4mm_P1.27mm
- U5, U6: footprint (none) -> Package_SO:SOP-20_7.5x12.8mm_P1.27mm
Changed lines of the file:
@@
 F 0 "U4" H 3300 4100 50  0000 C CNN
 F 1 "74HC595" H 3400 2800 50  0000 C CNN
-F 2 "" H 3150 3500 50  0001 C CNN
+F 2 "Package_SO:SOP-16_4.4x10.4mm_P1.27mm" H 3150 3500 50  0001 C CNN
 F 3 "http://www.ti.com/lit/ds/symlink/sn74hc595.pdf" H 3150 3500 50  0001 C CNN
 	1    3150 3500
@@
 F 0 "U5" H 6250 2450 50  0000 L CNN
 F 1 "L293DD" H 5650 3150 50  0000 L CNN
-F 2 "" H 5950 2600 50  0001 C CNN
+F 2 "Package_SO:SOP-20_7.5x12.8mm_P1.27mm" H 5950 2600 50  0001 C CNN
 F 3 "" H 5950 2600 50  0001 C CNN
 	1    5950 2750
@@
 F 0 "U5" H 8400 2450 50  0000 L CNN
 F 1 "L293DD" H 7800 3150 50  0000 L CNN
-F 2 "" H 8100 2600 50  0001 C CNN
+F 2 "Package_SO:SOP-20_7.5x12.8mm_P1.27mm" H 8100 2600 50  0001 C CNN
 F 3 "" H 8100 2600 50  0001 C CNN
 	2    8100 2750
@@
 F 0 "U6" H 6250 4300 50  0000 L CNN
 F 1 "L293DD" H 5650 5000 50  0000 L CNN
-F 2 "" H 5950 4450 50  0001 C CNN
+F 2 "Package_SO:SOP-20_7.5x12.8mm_P1.27mm" H 5950 4450 50  0001 C CNN
 F 3 "" H 5950 4450 50  0001 C CNN
 	1    5950 4600
@@
 F 0 "U6" H 8400 4300 50  0000 L CNN
 F 1 "L293DD" H 7800 5000 50  0000 L CNN
-F 2 "" H 8100 4450 50  0001 C CNN
+F 2 "Package_SO:SOP-20_7.5x12.8mm_P1.27mm" H 8100 4450 50  0001 C CNN
 F 3 "" H 8100 4450 50  0001 C CNN
 	2    8100 4600
