File: er2_pcbv2.sch (KiCad schematic (older format))
At the start: 6 parts, among them P1 CONN_3X2, P10 CONN_5, P2 CONN_3X2, P3 CONN_13X2

Commit message: pcb: signal led resistor changed
Parts:
- R1: value 330R -> 1,5k
Changed lines of the file:
@@
 LIBS:memory
 LIBS:xilinx
-LIBS:special
 LIBS:microcontrollers
 LIBS:dsp
@@
 LIBS:contrib
 LIBS:valves
+LIBS:er2_pcbv2-cache
 LIBS:linear2
 LIBS:xc6206
 LIBS:mma7455
 LIBS:l293dd
-EELAYER 27 0
+EELAYER 25 0
 EELAYER END
 $Descr A4 11693 8268
@@
 	3650 4100 3700 4100
 Wire Wire Line
-	4700 4100 5000 4100
+	4600 4100 5000 4100
 $Comp
 L R R1
@@
 P 4450 4100
 F 0 "R1" V 4530 4100 40  0000 C CNN
-F 1 "330R" V 4457 4101 40  0000 C CNN
+F 1 "1,5k" V 4457 4101 40  0000 C CNN
 F 2 "~" V 4380 4100 30  0000 C CNN
 F 3 "~" H 4450 4100 30  0000 C CNN
@@
 $EndComp
 Wire Wire Line
-	4100 4100 4200 4100
+	4100 4100 4300 4100
 $Sheet
 S 6900 2450 1200 650

Commit message: pcb: refresh footprints, accelerometer deleted
Parts:
- D1: footprint ~ -> LEDs:LED_0805
- P1, P2: footprint ~ -> Pin_Headers:Pin_Header_Straight_2x03_Pitch2.00mm
- P3: footprint ~ -> Pin_Headers:Pin_Header_Straight_2x13
- P4: renamed from P10; footprint ~ -> Pin_Headers:Pin_Header_Straight_1x05
- R1: footprint ~ -> Resistors_SMD:R_0805_HandSoldering
Connections:
- wire segments 76 -> 74
Changed lines of the file:
@@
 LIBS:linear2
 LIBS:xc6206
-LIBS:mma7455
 LIBS:l293dd
 EELAYER 25 0
@@
 $Descr A4 11693 8268
 encoding utf-8
-Sheet 1 4
+Sheet 1 3
 Title "er2 controller pcb"
 Date "1 jul 2015"
@@
 F 0 "P3" H 5400 5100 60  0000 C CNN
 F 1 "CONN_13X2" V 5400 4400 50  0000 C CNN
-F 2 "~" H 5400 4400 60  0000 C CNN
+F 2 "Pin_Headers:Pin_Header_Straight_2x13" H 5400 4400 60  0001 C CNN
 F 3 "~" H 5400 4400 60  0000 C CNN
 	1    5400 4400
@@
 F 0 "D1" H 3900 4200 50  0000 C CNN
 F 1 "LED" H 3900 4000 50  0000 C CNN
-F 2 "~" H 3900 4100 60  0000 C CNN
+F 2 "LEDs:LED_0805" H 3900 4100 60  0000 C CNN
 F 3 "~" H 3900 4100 60  0000 C CNN
 	1    3900 4100
@@
 F 0 "R1" V 4530 4100 40  0000 C CNN
 F 1 "1,5k" V 4457 4101 40  0000 C CNN
-F 2 "~" V 4380 4100 30  0000 C CNN
+F 2 "Resistors_SMD:R_0805_HandSoldering" V 4380 4100 30  0001 C CNN
 F 3 "~" H 4450 4100 30  0000 C CNN
 	1    4450 4100
@@
 	6000 4350 6950 4350
 Wire Wire Line
-	5800 4500 6000 4500
-Wire Wire Line
 	6000 4500 6000 4450
 Wire Wire Line
@@
 Wire Wire Line
 	6300 3800 6300 3750
-$Sheet
-S 3550 2350 900  500
-U 556229D8
-F0 "Accelerometer" 50
-F1 "accelerometer.sch" 50
-F2 "SDA" I R 4450 2500 60
-F3 "SCL" I R 4450 2700 60
-$EndSheet
 NoConn ~ 5000 3800
 Wire Wire Line
 	4850 3900 5000 3900
-Wire Wire Line
-	4850 2500 4450 2500
-Wire Wire Line
-	4450 2700 4800 2700
-Wire Wire Line
-	4800 2700 4800 4000
 Wire Wire Line
 	4800 4000 5000 4000
@@
 F 0 "P1" H 3650 5750 50  0000 C CNN
 F 1 "CONN_3X2" V 3650 5550 40  0000 C CNN
-F 2 "~" H 3650 5500 60  0000 C CNN
+F 2 "Pin_Headers:Pin_Header_Straight_2x03_Pitch2.00mm" H 3650 5500 60  0001 C CNN
 F 3 "~" H 3650 5500 60  0000 C CNN
 	1    3650 5500
@@
 F 0 "P2" H 3650 6400 50  0000 C CNN
 F 1 "CONN_3X2" V 3650 6200 40  0000 C CNN
-F 2 "~" H 3650 6150 60  0000 C CNN
+F 2 "Pin_Headers:Pin_Header_Straight_2x03_Pitch2.00mm" H 3650 6150 60  0001 C CNN
 F 3 "~" H 3650 6150 60  0000 C CNN
 	1    3650 6150
@@
 	5800 2800 5800 2900
 Wire Wire Line
-	5900 2800 5900 2950
+	5900 2950 5900 2800
 $Comp
 L +5V #PWR06
@@
 $EndComp
 $Comp
-L CONN_5 P10
+L CONN_5 P4
 U 1 1 55935FAC
 P 5800 2400
-F 0 "P10" V 5750 2400 50  0000 C CNN
+F 0 "P4" V 5750 2400 50  0000 C CNN
 F 1 "CONN_5" V 5850 2400 50  0000 C CNN
-F 2 "~" H 5800 2400 60  0000 C CNN
+F 2 "Pin_Headers:Pin_Header_Straight_1x05" H 5800 2400 60  0001 C CNN
 F 3 "~" H 5800 2400 60  0000 C CNN
 	1    5800 2400
@@
 $EndComp
 Wire Wire Line
-	4850 2500 4850 3900
-Wire Wire Line
 	5600 2800 5600 2850
 Wire Wire Line
@@
 Wire Wire Line
 	5800 2900 4800 2900
-Connection ~ 4800 2900
-Wire Wire Line
-	5900 2950 4850 2950
-Connection ~ 4850 2950
+Wire Wire Line
+	4850 2950 5900 2950
 Wire Wire Line
 	5700 2800 5700 3100
 NoConn ~ 6000 2800
+Wire Wire Line
+	5800 4500 6000 4500
+Wire Wire Line
+	4800 2900 4800 4000
+Wire Wire Line
+	4850 2950 4850 3900
 $EndSCHEMATC

Commit message: pcb: mma7455l replaced by mpu6050
Parts:
- D1: footprint LEDs:LED_0805 -> (none)
Connections:
- net labels added: +3.3V
- wire segments 74 -> 80
- no-connect marks 10 -> 9
Changed lines of the file:
@@
 LIBS:xc6206
 LIBS:l293dd
+LIBS:mpu-6050
 EELAYER 25 0
 EELAYER END
 $Descr A4 11693 8268
 encoding utf-8
-Sheet 1 3
+Sheet 1 4
 Title "er2 controller pcb"
-Date "1 jul 2015"
+Date "2016-06-28"
 Rev ""
 Comp "Institute for Mathematics, Mechanics, and Computer Science in the name of I.I. Vorovich"
@@
 Text Notes 5050 3500 0    60   ~ 0
   Raspberry PI\nGPIO connector
-$Comp
-L GND #PWR01
-U 1 1 553FB7B8
-P 6300 4100
-F 0 "#PWR01" H 6300 4100 30  0001 C CNN
-F 1 "GND" H 6300 4030 30  0001 C CNN
-F 2 "" H 6300 4100 60  0000 C CNN
-F 3 "" H 6300 4100 60  0000 C CNN
-	1    6300 4100
-	1    0    0    -1
-$EndComp
 NoConn ~ 5000 4600
 NoConn ~ 5000 5000
@@
 NoConn ~ 5800 3900
 NoConn ~ 5000 4200
-$Comp
-L LED D1
-U 1 1 554955EA
-P 3900 4100
-F 0 "D1" H 3900 4200 50  0000 C CNN
-F 1 "LED" H 3900 4000 50  0000 C CNN
-F 2 "LEDs:LED_0805" H 3900 4100 60  0000 C CNN
-F 3 "~" H 3900 4100 60  0000 C CNN
-	1    3900 4100
-	-1   0    0    1
-$EndComp
-$Comp
-L GND #PWR02
-U 1 1 554955F0
-P 3650 4400
-F 0 "#PWR02" H 3650 4400 30  0001 C CNN
-F 1 "GND" H 3650 4330 30  0001 C CNN
-F 2 "" H 3650 4400 60  0000 C CNN
-F 3 "" H 3650 4400 60  0000 C CNN
-	1    3650 4400
-	1    0    0    -1
-$EndComp
-Wire Wire Line
-	3650 4400 3650 4100
-Wire Wire Line
-	3650 4100 3700 4100
-Wire Wire Line
-	4600 4100 5000 4100
+Wire Wire Line
+	3050 4400 3050 4100
+Wire Wire Line
+	3050 4100 3100 4100
+Wire Wire Line
+	4000 4100 5000 4100
 $Comp
 L R R1
 U 1 1 5549595B
-P 4450 4100
-F 0 "R1" V 4530 4100 40  0000 C CNN
-F 1 "1,5k" V 4457 4101 40  0000 C CNN
-F 2 "Resistors_SMD:R_0805_HandSoldering" V 4380 4100 30  0001 C CNN
-F 3 "~" H 4450 4100 30  0000 C CNN
-	1    4450 4100
+P 3850 4100
+F 0 "R1" V 3930 4100 40  0000 C CNN
+F 1 "1,5k" V 3857 4101 40  0000 C CNN
+F 2 "Resistors_SMD:R_0805_HandSoldering" V 3780 4100 30  0001 C CNN
+F 3 "~" H 3850 4100 30  0000 C CNN
+	1    3850 4100
 	0    -1   -1   0
 $EndComp
 Wire Wire Line
-	4100 4100 4300 4100
+	3500 4100 3700 4100
 $Sheet
-S 6900 2450 1200 650
+S 7050 2850 850  350
 U 5561E615
 F0 "Power supply" 50
@@
 Wire Wire Line
 	4650 4300 5000 4300
-$Comp
-L +5V #PWR03
-U 1 1 55621EDD
-P 6300 3750
-F 0 "#PWR03" H 6300 3840 20  0001 C CNN
-F 1 "+5V" H 6300 3840 30  0000 C CNN
-F 2 "" H 6300 3750 60  0000 C CNN
-F 3 "" H 6300 3750 60  0000 C CNN
-	1    6300 3750
-	1    0    0    -1
-$EndComp
-Wire Wire Line
-	5800 3800 6300 3800
-Wire Wire Line
-	6300 3800 6300 3750
-NoConn ~ 5000 3800
-Wire Wire Line
-	4850 3900 5000 3900
-Wire Wire Line
-	4800 4000 5000 4000
+Wire Wire Line
+	4400 3900 5000 3900
+Wire Wire Line
+	4350 4000 5000 4000
 $Comp
 L CONN_3X2 P1
@@
 Wire Wire Line
 	3050 5350 3250 5350
-$Comp
-L GND #PWR04
-U 1 1 5591E894
-P 3050 6600
-F 0 "#PWR04" H 3050 6600 30  0001 C CNN
-F 1 "GND" H 3050 6530 30  0001 C CNN
-F 2 "" H 3050 6600 60  0000 C CNN
-F 3 "" H 3050 6600 60  0000 C CNN
-	1    3050 6600
-	1    0    0    -1
-$EndComp
 Connection ~ 3050 6000
 Wire Wire Line
@@
 Wire Wire Line
 	4050 5350 4400 5350
-$Comp
-L +5V #PWR05
-U 1 1 5591EF25
-P 4400 5200
-F 0 "#PWR05" H 4400 5290 20  0001 C CNN
-F 1 "+5V" H 4400 5290 30  0000 C CNN
-F 2 "" H 4400 5200 60  0000 C CNN
-F 3 "" H 4400 5200 60  0000 C CNN
-	1    4400 5200
-	1    0    0    -1
-$EndComp
 Wire Wire Line
 	4400 5350 4400 5200
@@
 	4300 5600 4300 6200
 Wire Wire Line
-	5800 2800 5800 2900
-Wire Wire Line
-	5900 2950 5900 2800
-$Comp
-L +5V #PWR06
+	5800 2900 5800 2800
+Wire Wire Line
+	5900 3000 5900 2800
+$Comp
+L +5V #PWR01
 U 1 1 55935D38
 P 5450 2550
-F 0 "#PWR06" H 5450 2640 20  0001 C CNN
+F 0 "#PWR01" H 5450 2640 20  0001 C CNN
 F 1 "+5V" H 5450 2640 30  0000 C CNN
 F 2 "" H 5450 2550 60  0000 C CNN
@@
 Wire Wire Line
 	5450 2550 5450 2850
-$Comp
-L GND #PWR07
-U 1 1 55935E4C
-P 5700 3100
-F 0 "#PWR07" H 5700 3100 30  0001 C CNN
-F 1 "GND" H 5700 3030 30  0001 C CNN
-F 2 "" H 5700 3100 60  0000 C CNN
-F 3 "" H 5700 3100 60  0000 C CNN
-	1    5700 3100
-	1    0    0    -1
-$EndComp
 $Comp
 L CONN_5 P4
@@
 	5600 2850 5450 2850
 Wire Wire Line
-	5800 2900 4800 2900
-Wire Wire Line
-	4850 2950 5900 2950
-Wire Wire Line
 	5700 2800 5700 3100
 NoConn ~ 6000 2800
 Wire Wire Line
 	5800 4500 6000 4500
-Wire Wire Line
-	4800 2900 4800 4000
-Wire Wire Line
-	4850 2950 4850 3900
+$Sheet
+S 3200 2800 850  600
+U 5771B746
+F0 "mpu6050" 60
+F1 "mpu6050.sch" 60
+F2 "SCL" I R 4050 3300 60
+F3 "SDA" I R 4050 3200 60
+F4 "AUX_CL" O R 4050 2900 60
+F5 "AUX_DA" O R 4050 3000 60
+$EndSheet
+Wire Wire Line
+	4050 3200 4400 3200
+Wire Wire Line
+	4050 3000 5900 3000
+Wire Wire Line
+	4350 3300 4050 3300
+Wire Wire Line
+	4050 2900 5800 2900
+$Comp
+L +3.3V #PWR02
+U 1 1 5772964F
+P 4700 3400
+F 0 "#PWR02" H 4700 3250 50  0001 C CNN
+F 1 "+3.3V" H 4700 3540 50  0000 C CNN
+F 2 "" H 4700 3400 50  0000 C CNN
+F 3 "" H 4700 3400 50  0000 C CNN
+	1    4700 3400
+	1    0    0    -1
+$EndComp
+Wire Wire Line
+	4350 4000 4350 3300
+Wire Wire Line
+	4400 3200 4400 3900
+Wire Wire Line
+	5800 3800 5950 3800
+Wire Wire Line
+	5950 3800 5950 3750
+$Comp
+L +5V #PWR03
+U 1 1 5772A0A4
+P 5950 3750
+F 0 "#PWR03" H 5950 3600 50  0001 C CNN
+F 1 "+5V" H 5950 3890 50  0000 C CNN
+F 2 "" H 5950 3750 50  0000 C CNN
+F 3 "" H 5950 3750 50  0000 C CNN
+	1    5950 3750
+	1    0    0    -1
+$EndComp
+$Comp
+L GND #PWR04
+U 1 1 5772B1EE
+P 5700 3100
+F 0 "#PWR04" H 5700 2850 50  0001 C CNN
+F 1 "GND" H 5700 2950 50  0000 C CNN
+F 2 "" H 5700 3100 50  0000 C CNN
+F 3 "" H 5700 3100 50  0000 C CNN
+	1    5700 3100
+	1    0    0    -1
+$EndComp
+$Comp
+L GND #PWR05
+U 1 1 5772B2F0
+P 3050 6600
+F 0 "#PWR05" H 3050 6350 50  0001 C CNN
+F 1 "GND" H 3050 6450 50  0000 C CNN
+F 2 "" H 3050 6600 50  0000 C CNN
+F 3 "" H 3050 6600 50  0000 C CNN
+	1    3050 6600
+	1    0    0    -1
+$EndComp
+$Comp
+L +5V #PWR06
+U 1 1 5772B72C
+P 4400 5200
+F 0 "#PWR06" H 4400 5050 50  0001 C CNN
+F 1 "+5V" H 4400 5340 50  0000 C CNN
+F 2 "" H 4400 5200 50  0000 C CNN
+F 3 "" H 4400 5200 50  0000 C CNN
+	1    4400 5200
+	1    0    0    -1
+$EndComp
+$Comp
+L GND #PWR07
+U 1 1 5772B8F1
+P 3050 4400
+F 0 "#PWR07" H 3050 4150 50  0001 C CNN
+F 1 "GND" H 3050 4250 50  0000 C CNN
+F 2 "" H 3050 4400 50  0000 C CNN
+F 3 "" H 3050 4400 50  0000 C CNN
+	1    3050 4400
+	1    0    0    -1
+$EndComp
+$Comp
+L LED D1
+U 1 1 5772B970
+P 3300 4100
+F 0 "D1" H 3300 4200 50  0000 C CNN
+F 1 "LED" H 3300 4000 50  0000 C CNN
+F 2 "" H 3300 4100 50  0000 C CNN
+F 3 "" H 3300 4100 50  0000 C CNN
+	1    3300 4100
+	-1   0    0    1
+$EndComp
+$Comp
+L PWR_FLAG #FLG08
+U 1 1 5772E95B
+P 4700 3600
+F 0 "#FLG08" H 4700 3695 50  0001 C CNN
+F 1 "PWR_FLAG" H 4700 3780 50  0000 C CNN
+F 2 "" H 4700 3600 50  0000 C CNN
+F 3 "" H 4700 3600 50  0000 C CNN
+	1    4700 3600
+	-1   0    0    1
+$EndComp
+Wire Wire Line
+	4700 3600 4700 3400
+Wire Wire Line
+	4700 3500 4950 3500
+Wire Wire Line
+	4950 3500 4950 3800
+Wire Wire Line
+	4950 3800 5000 3800
+Connection ~ 4700 3500
+$Comp
+L GND #PWR09
+U 1 1 5772F7CC
+P 6300 4100
+F 0 "#PWR09" H 6300 3850 50  0001 C CNN
+F 1 "GND" H 6300 3950 50  0000 C CNN
+F 2 "" H 6300 4100 50  0000 C CNN
+F 3 "" H 6300 4100 50  0000 C CNN
+	1    6300 4100
+	1    0    0    -1
+$EndComp
 $EndSCHEMATC

Commit message: pcb: 74РС595 is conected SPI
Connections:
- wire segments 80 -> 78
- no-connect marks 9 -> 11
Changed lines of the file:
@@
 Title "er2 controller pcb"
 Date "2016-06-28"
-Rev ""
+Rev "2"
 Comp "Institute for Mathematics, Mechanics, and Computer Science in the name of I.I. Vorovich"
 Comment1 ""
@@
 	1    0    0    -1
 $EndComp
-Wire Wire Line
-	5800 4000 6300 4000
-Wire Wire Line
-	6300 4000 6300 4100
 Text Notes 5050 3500 0    60   ~ 0
   Raspberry PI\nGPIO connector
@@
 	8250 5250 4700 5250
 Wire Wire Line
-	4700 5250 4700 4400
-Wire Wire Line
-	4700 4400 5000 4400
-Wire Wire Line
 	8000 4450 8300 4450
 Wire Wire Line
@@
 Wire Wire Line
 	8300 5300 4650 5300
-Wire Wire Line
-	4650 5300 4650 4300
-Wire Wire Line
-	4650 4300 5000 4300
 Wire Wire Line
 	4400 3900 5000 3900
@@
 Wire Wire Line
 	4400 3200 4400 3900
-Wire Wire Line
-	5800 3800 5950 3800
-Wire Wire Line
-	5950 3800 5950 3750
 $Comp
 L +5V #PWR03
 U 1 1 5772A0A4
-P 5950 3750
-F 0 "#PWR03" H 5950 3600 50  0001 C CNN
-F 1 "+5V" H 5950 3890 50  0000 C CNN
-F 2 "" H 5950 3750 50  0000 C CNN
-F 3 "" H 5950 3750 50  0000 C CNN
-	1    5950 3750
+P 6100 3750
+F 0 "#PWR03" H 6100 3600 50  0001 C CNN
+F 1 "+5V" H 6100 3890 50  0000 C CNN
+F 2 "" H 6100 3750 50  0000 C CNN
+F 3 "" H 6100 3750 50  0000 C CNN
+	1    6100 3750
 	1    0    0    -1
 $EndComp
@@
 L GND #PWR09
 U 1 1 5772F7CC
-P 6300 4100
-F 0 "#PWR09" H 6300 3850 50  0001 C CNN
-F 1 "GND" H 6300 3950 50  0000 C CNN
-F 2 "" H 6300 4100 50  0000 C CNN
-F 3 "" H 6300 4100 50  0000 C CNN
-	1    6300 4100
-	1    0    0    -1
-$EndComp
+P 6100 4100
+F 0 "#PWR09" H 6100 3850 50  0001 C CNN
+F 1 "GND" H 6100 3950 50  0000 C CNN
+F 2 "" H 6100 4100 50  0000 C CNN
+F 3 "" H 6100 4100 50  0000 C CNN
+	1    6100 4100
+	1    0    0    -1
+$EndComp
+NoConn ~ 5000 4300
+Wire Wire Line
+	4700 5250 4700 4900
+Connection ~ 4700 4900
+Wire Wire Line
+	4650 5300 4650 4700
+Connection ~ 4650 4700
+NoConn ~ 5000 4400
+Wire Wire Line
+	5800 3800 6100 3800
+Wire Wire Line
+	6100 3800 6100 3750
+Wire Wire Line
+	5800 4000 6100 4000
+Wire Wire Line
+	6100 4000 6100 4100
 $EndSCHEMATC

Commit message: pcb: ADC PCF85911 batery control added
Parts:
- removed P1, P2: CONN_3X2, Pin_Headers:Pin_Header_Straight_2x03_Pitch2.00mm, symbol CONN_3X2
- removed P3: CONN_13X2, Pin_Headers:Pin_Header_Straight_2x13, symbol CONN_13X2
- removed P4: CONN_5, Pin_Headers:Pin_Header_Straight_1x05, symbol CONN_5
- added P1, P2: CONN_02X03, Pin_Headers:Pin_Header_Straight_2x03, symbol CONN_02X03
- added P3: CONN_02X13, Pin_Headers:Pin_Header_Straight_2x13, symbol CONN_02X13
- added P4: CONN_01X05, Pin_Headers:Pin_Header_Straight_1x05, symbol CONN_01X05
- D1: footprint (none) -> LEDs:LED_0805
Connections:
- wire segments 78 -> 79
