File: mpu6050.sch (KiCad schematic (older format))
At the start: 7 parts, among them U2 MPU-6050

Commit message: pcb: ADC PCF85911 batery control added
Parts:
- renumbered R11 to R15, R12 to R16, U2 to U3
Changed lines of the file:
@@
 $EndDescr
 $Comp
-L MPU-6050 U2
+L MPU-6050 U3
 U 1 1 5771B961
 P 5950 4000
-F 0 "U2" H 6300 3300 60  0000 C CNN
+F 0 "U3" H 6300 3300 60  0000 C CNN
 F 1 "MPU-6050" H 5700 3300 60  0000 C CNN
 F 2 "Housings_DFN_QFN:QFN-24-1EP_4x4mm_Pitch0.5mm" H 5950 3750 60  0001 C CNN
@@
 $EndComp
 $Comp
-L +3.3V #PWR037
+L +3.3V #PWR044
 U 1 1 57722230
 P 3800 3050
-F 0 "#PWR037" H 3800 2900 50  0001 C CNN
+F 0 "#PWR044" H 3800 2900 50  0001 C CNN
 F 1 "+3.3V" H 3800 3190 50  0000 C CNN
 F 2 "" H 3800 3050 50  0000 C CNN
@@
 $EndComp
 $Comp
-L GND #PWR038
+L GND #PWR045
 U 1 1 57722246
 P 3800 3950
-F 0 "#PWR038" H 3800 3700 50  0001 C CNN
+F 0 "#PWR045" H 3800 3700 50  0001 C CNN
 F 1 "GND" H 3800 3800 50  0000 C CNN
 F 2 "" H 3800 3950 50  0000 C CNN
@@
 $EndComp
 $Comp
-L GND #PWR039
+L GND #PWR046
 U 1 1 57722361
 P 4700 3950
-F 0 "#PWR039" H 4700 3700 50  0001 C CNN
+F 0 "#PWR046" H 4700 3700 50  0001 C CNN
 F 1 "GND" H 4700 3800 50  0000 C CNN
 F 2 "" H 4700 3950 50  0000 C CNN
@@
 $EndComp
 $Comp
-L GND #PWR040
+L GND #PWR047
 U 1 1 57722508
 P 4400 3950
-F 0 "#PWR040" H 4400 3700 50  0001 C CNN
+F 0 "#PWR047" H 4400 3700 50  0001 C CNN
 F 1 "GND" H 4400 3800 50  0000 C CNN
 F 2 "" H 4400 3950 50  0000 C CNN
@@
 	4400 3450 5150 3450
 $Comp
-L GND #PWR041
+L GND #PWR048
 U 1 1 577225CD
 P 5000 3950
-F 0 "#PWR041" H 5000 3700 50  0001 C CNN
+F 0 "#PWR048" H 5000 3700 50  0001 C CNN
 F 1 "GND" H 5000 3800 50  0000 C CNN
 F 2 "" H 5000 3950 50  0000 C CNN
@@
 	3800 3050 3800 3650
 $Comp
-L GND #PWR042
+L GND #PWR049
 U 1 1 57722D08
 P 6900 4200
-F 0 "#PWR042" H 6900 3950 50  0001 C CNN
+F 0 "#PWR049" H 6900 3950 50  0001 C CNN
 F 1 "GND" H 6900 4050 50  0000 C CNN
 F 2 "" H 6900 4200 50  0000 C CNN
@@
 	6900 3800 6900 4200
 $Comp
-L R R11
+L R R15
 U 1 1 57722D56
 P 7000 2950
-F 0 "R11" V 7080 2950 50  0000 C CNN
+F 0 "R15" V 7080 2950 50  0000 C CNN
 F 1 "10k" V 7000 2950 50  0000 C CNN
 F 2 "Resistors_SMD:R_0805_HandSoldering" V 6930 2950 50  0001 C CNN
@@
 $EndComp
 $Comp
-L R R12
+L R R16
 U 1 1 57722DD3
 P 7200 2950
-F 0 "R12" V 7280 2950 50  0000 C CNN
+F 0 "R16" V 7280 2950 50  0000 C CNN
 F 1 "10k" V 7200 2950 50  0000 C CNN
 F 2 "Resistors_SMD:R_0805_HandSoldering" V 7130 2950 50  0001 C CNN
@@
 $EndComp
 $Comp
-L +3.3V #PWR043
+L +3.3V #PWR050
 U 1 1 57722E0B
 P 7100 2700
-F 0 "#PWR043" H 7100 2550 50  0001 C CNN
+F 0 "#PWR050" H 7100 2550 50  0001 C CNN
 F 1 "+3.3V" H 7100 2840 50  0000 C CNN
 F 2 "" H 7100 2700 50  0000 C CNN
@@
 $EndComp
 $Comp
-L GND #PWR044
+L GND #PWR051
 U 1 1 57728850
 P 4100 3950
-F 0 "#PWR044" H 4100 3700 50  0001 C CNN
+F 0 "#PWR051" H 4100 3700 50  0001 C CNN
 F 1 "GND" H 4100 3800 50  0000 C CNN
 F 2 "" H 4100 3950 50  0000 C CNN
