File: power_supply.sch (KiCad schematic (older format))
At the start: 12 parts, among them IC1 LM2596S, IC2 XC6206, P4 CONN_2, P5 CONN_2

Commit message: pcb: refresh footprints, accelerometer deleted
Parts:
- removed C3, C4: 1uF, ~, symbol C
- added C3, C4: 1uF, Capacitors_SMD:C_0805_HandSoldering, symbol C_Small
- C1: footprint ~ -> Capacitors_SMD:c_elec_6.3x5.7
- C2: footprint ~ -> Capacitors_SMD:c_elec_6.3x7.7
- D2: footprint ~ -> Diodes_SMD:SMC_Handsoldering
- D3: footprint ~ -> LEDs:LED_0805
- IC1: footprint linear2-TO263-5 -> TO_SOT_Packages_SMD:TO-263-5Lead
- IC2: footprint ~ -> TO_SOT_Packages_SMD:SOT-23
- L1: footprint ~ -> Inductors:Inductor_1212
- P5: renamed from P4; footprint ~ -> (none)
- P6: renamed from P5; footprint ~ -> (none)
- R2: value 330R -> 1.5k; footprint ~ -> Resistors_SMD:R_0805_HandSoldering
Changed lines of the file:
@@
 LIBS:linear2
 LIBS:xc6206
-LIBS:mma7455
 LIBS:l293dd
 EELAYER 25 0
@@
 $Descr A4 11693 8268
 encoding utf-8
-Sheet 2 4
+Sheet 2 3
 Title ""
 Date "1 jul 2015"
@@
 F 0 "D2" H 5050 4750 40  0000 C CNN
 F 1 "1N5822" H 5050 4550 40  0000 C CNN
-F 2 "~" H 5050 4650 60  0000 C CNN
+F 2 "Diodes_SMD:SMC_Handsoldering" H 5050 4650 60  0000 C CNN
 F 3 "~" H 5050 4650 60  0000 C CNN
 	1    5050 4650
@@
 F 0 "L1" V 5500 4350 40  0000 C CNN
 F 1 "33uH" V 5650 4350 40  0000 C CNN
-F 2 "~" H 5550 4350 60  0000 C CNN
+F 2 "Inductors:Inductor_1212" H 5550 4350 60  0001 C CNN
 F 3 "~" H 5550 4350 60  0000 C CNN
 	1    5550 4350
@@
 F 0 "IC1" H 3950 4500 50  0000 L BNN
 F 1 "LM2596S" H 4350 4500 50  0000 L BNN
-F 2 "linear2-TO263-5" H 4250 4400 50  0001 C CNN
+F 2 "TO_SOT_Packages_SMD:TO-263-5Lead" H 4250 4400 50  0001 C CNN
 F 3 "" H 4250 4250 60  0000 C CNN
 	1    4250 4250
@@
 Connection ~ 5050 4350
 Wire Wire Line
-	6050 4150 6050 4450
+	6050 4150 6050 4500
 Wire Wire Line
 	4650 4150 6050 4150
 Connection ~ 6050 4350
 Wire Wire Line
-	6050 5000 6050 4850
+	6050 4800 6050 5000
 $Comp
 L GND #PWR011
@@
 	5050 4850 5050 5000
 Wire Wire Line
-	3600 4450 3600 4350
+	3600 4350 3600 4500
 Wire Wire Line
 	3300 4350 3850 4350
@@
 $EndComp
 Wire Wire Line
-	3600 5000 3600 4850
+	3600 4800 3600 5000
 Wire Wire Line
 	3300 4300 3300 4400
@@
 F 0 "C1" H 3650 4750 50  0000 L CNN
 F 1 "100uF" H 3650 4550 50  0000 L CNN
-F 2 "~" H 3600 4650 60  0000 C CNN
+F 2 "Capacitors_SMD:c_elec_6.3x5.7" H 3600 4650 60  0000 C CNN
 F 3 "~" H 3600 4650 60  0000 C CNN
 	1    3600 4650
@@
 F 0 "C2" H 6100 4750 50  0000 L CNN
 F 1 "220uF" H 6100 4550 50  0000 L CNN
-F 2 "~" H 6050 4650 60  0000 C CNN
+F 2 "Capacitors_SMD:c_elec_6.3x7.7" H 6050 4650 60  0000 C CNN
 F 3 "~" H 6050 4650 60  0000 C CNN
 	1    6050 4650
@@
 Connection ~ 3300 4350
 Text Notes 5000 3800 0    60   ~ 0
-Switched-mode \npower supply\n(12V -> 5V)\n(5V   -> 3.3V)
+Switched-mode \npower supply\n(12V -> 5V)\n(5V  -> 3.3V)
 $Comp
 L R R2
@@
 P 6200 3900
 F 0 "R2" V 6280 3900 40  0000 C CNN
-F 1 "330R" V 6207 3901 40  0000 C CNN
-F 2 "~" V 6130 3900 30  0000 C CNN
+F 1 "1.5k" V 6207 3901 40  0000 C CNN
+F 2 "Resistors_SMD:R_0805_HandSoldering" V 6130 3900 30  0001 C CNN
 F 3 "~" H 6200 3900 30  0000 C CNN
 	1    6200 3900
@@
 F 0 "D3" H 6500 3650 50  0000 C CNN
 F 1 "LED" H 6500 3450 50  0000 C CNN
-F 2 "~" H 6500 3550 60  0000 C CNN
+F 2 "LEDs:LED_0805" H 6500 3550 60  0000 C CNN
 F 3 "~" H 6500 3550 60  0000 C CNN
 	1    6500 3550
@@
 $EndComp
 Wire Wire Line
-	6200 3650 6200 3550
+	6200 3550 6200 3750
 Wire Wire Line
 	6200 3550 6300 3550
 Wire Wire Line
-	6200 4150 6200 4350
+	6200 4050 6200 4350
 Connection ~ 6200 4350
 $Comp
@@
 F 0 "IC2" H 7150 4700 60  0000 C CNN
 F 1 "XC6206" H 7350 4250 60  0000 C CNN
-F 2 "~" H 7150 4450 60  0000 C CNN
+F 2 "TO_SOT_Packages_SMD:SOT-23" H 7150 4450 60  0001 C CNN
 F 3 "~" H 7150 4450 60  0000 C CNN
 	1    7150 4450
@@
 Wire Wire Line
 	5850 4350 6850 4350
-$Comp
-L C C3
-U 1 1 5561E74D
-P 6700 4700
-F 0 "C3" H 6700 4800 40  0000 L CNN
-F 1 "1uF" H 6706 4615 40  0000 L CNN
-F 2 "~" H 6738 4550 30  0000 C CNN
-F 3 "~" H 6700 4700 60  0000 C CNN
-	1    6700 4700
-	1    0    0    -1
-$EndComp
-$Comp
-L C C4
-U 1 1 5561E753
-P 7700 4700
-F 0 "C4" H 7700 4800 40  0000 L CNN
-F 1 "1uF" H 7706 4615 40  0000 L CNN
-F 2 "~" H 7738 4550 30  0000 C CNN
-F 3 "~" H 7700 4700 60  0000 C CNN
-	1    7700 4700
-	1    0    0    -1
-$EndComp
 Connection ~ 7700 4350
 Wire Wire Line
-	6700 4350 6700 4500
+	6700 4350 6700 4600
 Connection ~ 6700 4350
 $Comp
@@
 $EndComp
 Wire Wire Line
-	7700 4900 7700 5000
-Wire Wire Line
-	6700 4900 6700 5000
-Wire Wire Line
-	7700 4500 7700 4350
-$Comp
-L CONN_2 P5
+	7700 4800 7700 5000
+Wire Wire Line
+	6700 4800 6700 5000
+Wire Wire Line
+	7700 4350 7700 4600
+$Comp
+L CONN_2 P6
 U 1 1 5561E9D1
 P 8050 2400
-F 0 "P5" V 8000 2400 40  0000 C CNN
+F 0 "P6" V 8000 2400 40  0000 C CNN
 F 1 "CONN_2" V 8100 2400 40  0000 C CNN
-F 2 "~" H 8050 2400 60  0000 C CNN
+F 2 "" H 8050 2400 60  0001 C CNN
 F 3 "~" H 8050 2400 60  0000 C CNN
 	1    8050 2400
@@
 $EndComp
 $Comp
-L CONN_2 P4
+L CONN_2 P5
 U 1 1 5561E9E3
 P 5600 2400
-F 0 "P4" V 5550 2400 40  0000 C CNN
+F 0 "P5" V 5550 2400 40  0000 C CNN
 F 1 "CONN_2" V 5650 2400 40  0000 C CNN
-F 2 "~" H 5600 2400 60  0000 C CNN
+F 2 "" H 5600 2400 60  0001 C CNN
 F 3 "~" H 5600 2400 60  0000 C CNN
 	1    5600 2400
@@
 	8050 4350 8050 4200
 $Comp
+L C_Small C3
+U 1 1 5771DFF7
+P 6700 4700
+F 0 "C3" H 6710 4770 50  0000 L CNN
+F 1 "1uF" H 6710 4620 50  0000 L CNN
+F 2 "Capacitors_SMD:C_0805_HandSoldering" H 6700 4700 50  0001 C CNN
+F 3 "" H 6700 4700 50  0000 C CNN
+	1    6700 4700
+	1    0    0    -1
+$EndComp
+$Comp
+L C_Small C4
+U 1 1 5771E07B
+P 7700 4700
+F 0 "C4" H 7710 4770 50  0000 L CNN
+F 1 "1uF" H 7710 4620 50  0000 L CNN
+F 2 "Capacitors_SMD:C_0805_HandSoldering" H 7700 4700 50  0001 C CNN
+F 3 "" H 7700 4700 50  0000 C CNN
+	1    7700 4700
+	1    0    0    -1
+$EndComp
+$Comp
 L PWR_FLAG #FLG025
-U 1 1 5561EDF3
-P 7450 2600
-F 0 "#FLG025" H 7450 2695 30  0001 C CNN
-F 1 "PWR_FLAG" H 7450 2780 30  0000 C CNN
-F 2 "" H 7450 2600 60  0000 C CNN
-F 3 "" H 7450 2600 60  0000 C CNN
-	1    7450 2600
+U 1 1 5772005F
+P 7500 2650
+F 0 "#FLG025" H 7500 2745 50  0001 C CNN
+F 1 "PWR_FLAG" H 7500 2830 50  0000 C CNN
+F 2 "" H 7500 2650 50  0000 C CNN
+F 3 "" H 7500 2650 50  0000 C CNN
+	1    7500 2650
 	-1   0    0    1
 $EndComp
 Wire Wire Line
-	7450 2600 7450 2500
-Connection ~ 7450 2500
+	7500 2650 7500 2500
+Connection ~ 7500 2500
 $EndSCHEMATC

Commit message: pcb: RPi power supply deleted
Parts:
- removed P5: CONN_2, symbol CONN_2
Connections:
- wire segments 39 -> 35
Other:
- note removed: "Raspberry PI\npower supply\nvoltage (+5V)"
Changed lines of the file:
@@
-	1    0    0    -1
-$EndComp
-$Comp
-L CONN_2 P5
-U 1 1 5561E9E3
-P 5600 2400
-F 0 "P5" V 5550 2400 40  0000 C CNN
-F 1 "CONN_2" V 5650 2400 40  0000 C CNN
-F 2 "" H 5600 2400 60  0001 C CNN
-F 3 "~" H 5600 2400 60  0000 C CNN
-	1    5600 2400
-	1    0    0    -1
-$EndComp
-$Comp
-L GND #PWR023
-U 1 1 5561E9E9
-P 5150 2700
-F 0 "#PWR023" H 5150 2700 30  0001 C CNN
-F 1 "GND" H 5150 2630 30  0001 C CNN
-F 2 "" H 5150 2700 60  0000 C CNN
-F 3 "" H 5150 2700 60  0000 C CNN
-	1    5150 2700
 	1    0    0    -1
 $EndComp
@@
 Wire Wire Line
 	7150 2300 7700 2300
-Wire Wire Line
-	5150 2150 5150 2300
-Wire Wire Line
-	5150 2300 5250 2300
 Text Notes 8200 2400 0    60   ~ 0
 Power supply\nvoltage (+12V)
-Text Notes 5750 2350 0    60   ~ 0
-Raspberry PI\npower supply\nvoltage (+5V)
-$Comp
-L +5V #PWR024
-U 1 1 5561E9F6
-P 5150 2150
-F 0 "#PWR024" H 5150 2240 20  0001 C CNN
-F 1 "+5V" H 5150 2240 30  0000 C CNN
-F 2 "" H 5150 2150 60  0000 C CNN
-F 3 "" H 5150 2150 60  0000 C CNN
-	1    5150 2150
-	1    0    0    -1
-$EndComp
-Wire Wire Line
-	5250 2500 5150 2500
-Wire Wire Line
-	5150 2500 5150 2700
 Wire Wire Line
 	7150 2500 7150 2700

Commit message: pcb: mma7455l replaced by mpu6050
Parts:
- removed C3, C4: 1uF, Capacitors_SMD:C_0805_HandSoldering, symbol C_Small
- removed IC2: XC6206, TO_SOT_Packages_SMD:SOT-23, symbol XC6206
- renumbered P6 to P5
Connections:
- net labels removed: +3.3V
- wire segments 35 -> 26
Other:
- note added: "Switched-mode \npower supply\n(12V -> 5V)"
- note removed: "Switched-mode \npower supply\n(12V -> 5V)\n(5V -> 3.3V)"

Commit message: pcb: ADC PCF85911 batery control added
Parts:
- removed C1: 100uF, Capacitors_SMD:c_elec_6.3x5.7, symbol CP1
- removed C2: 220uF, Capacitors_SMD:c_elec_6.3x7.7, symbol CP1
- removed D2: 1N5822, Diodes_SMD:SMC_Handsoldering, symbol DIODESCH
- removed P5: CONN_2, symbol CONN_2
- added C1: 100uF, Capacitors_SMD:c_elec_6.3x5.3, symbol CP
- added C2: 220uF, Capacitors_SMD:c_elec_6.3x7.7, symbol CP
- added D2: 1N5822, Diodes_SMD:SMC_Handsoldering, symbol D_Schottky
- added P5: CONN_01X04, Connectors_JST:JST_XH_B04B-XH-A_04x2.50mm_Straight, symbol CONN_01X04
- added R3, R4, R6: 10k, Resistors_SMD:R_0805_HandSoldering, symbol R
- added R5: 20k, Resistors_SMD:R_0805_HandSoldering, symbol R
- added U1: PCF8591, SMD_Packages:SO-16-W, symbol PCF8591
Connections:
- net labels added: SCL, SDA
- wire segments 26 -> 52
- no-connect marks 0 -> 3
Other:
- note added: "ADC\nBattery control"

Commit message: pcb layout added
Parts:
- D2: footprint Diodes_SMD:SMC_Handsoldering -> Diodes_SMD:SOD-123
Changed lines of the file:
@@
 F 0 "D2" H 3700 5450 50  0000 C CNN
 F 1 "1N5822" H 3700 5250 50  0000 C CNN
-F 2 "Diodes_SMD:SMC_Handsoldering" H 3700 5350 50  0001 C CNN
+F 2 "Diodes_SMD:SOD-123" H 3700 5350 50  0001 C CNN
 F 3 "" H 3700 5350 50  0000 C CNN
 	1    3700 5350

Commit message: power supply 12V connector added
Parts:
- added P10: CONN_01X02, Pin_Headers:Pin_Header_Straight_1x02, symbol CONN_01X02
Connections:
- wire segments 52 -> 56
Other:
- note added: "Balancing battery\n connector"
Changed lines of the file:
@@
 LIBS:contrib
 LIBS:valves
-LIBS:er2_pcbv2-cache
 LIBS:linear2
 LIBS:xc6206
@@
 	0    1    1    0
 $EndComp
-Text Notes 4600 2000 0    60   ~ 0
+Text Notes 3000 2100 0    60   ~ 0
 Power supply\nvoltage (+12V)
 $Comp
 L PWR_FLAG #FLG010
 U 1 1 5772005F
-P 6150 2300
-F 0 "#FLG010" H 6150 2395 50  0001 C CNN
-F 1 "PWR_FLAG" H 6150 2480 50  0000 C CNN
-F 2 "" H 6150 2300 50  0000 C CNN
-F 3 "" H 6150 2300 50  0000 C CNN
-	1    6150 2300
+P 3650 2800
+F 0 "#FLG010" H 3650 2895 50  0001 C CNN
+F 1 "PWR_FLAG" H 3650 2980 50  0000 C CNN
+F 2 "" H 3650 2800 50  0000 C CNN
+F 3 "" H 3650 2800 50  0000 C CNN
+	1    3650 2800
 	-1   0    0    1
 $EndComp
@@
 L +12V #PWR013
 U 1 1 5772AAB6
-P 6150 2100
-F 0 "#PWR013" H 6150 1950 50  0001 C CNN
-F 1 "+12V" H 6150 2240 50  0000 C CNN
-F 2 "" H 6150 2100 50  0000 C CNN
-F 3 "" H 6150 2100 50  0000 C CNN
-	1    6150 2100
+P 6000 2250
+F 0 "#PWR013" H 6000 2100 50  0001 C CNN
+F 1 "+12V" H 6000 2390 50  0000 C CNN
+F 2 "" H 6000 2250 50  0000 C CNN
+F 3 "" H 6000 2250 50  0000 C CNN
+	1    6000 2250
 	1    0    0    -1
 $EndComp
@@
 L GND #PWR014
 U 1 1 5772AECD
-P 5300 2400
-F 0 "#PWR014" H 5300 2150 50  0001 C CNN
-F 1 "GND" H 5300 2250 50  0000 C CNN
-F 2 "" H 5300 2400 50  0000 C CNN
-F 3 "" H 5300 2400 50  0000 C CNN
-	1    5300 2400
+P 5550 2300
+F 0 "#PWR014" H 5550 2050 50  0001 C CNN
+F 1 "GND" H 5550 2150 50  0000 C CNN
+F 2 "" H 5550 2300 50  0000 C CNN
+F 3 "" H 5550 2300 50  0000 C CNN
+	1    5550 2300
 	1    0    0    -1
 $EndComp
@@
 $EndComp
 Wire Wire Line
-	5550 2100 5550 2350
-Wire Wire Line
 	5850 2100 5850 2800
-Wire Wire Line
-	5850 2200 6150 2200
-Wire Wire Line
-	6150 2100 6150 2300
-Connection ~ 6150 2200
 $Comp
 L PCF8591 U1
@@
 Wire Wire Line
 	5750 2100 5750 3000
-Connection ~ 5850 2200
 Wire Wire Line
 	5750 3000 5950 3000
@@
 	1950 5600 1950 5450
 Connection ~ 1950 5000
-$Comp
-L PWR_FLAG #FLG027
-U 1 1 5773E5B0
-P 5300 2300
-F 0 "#FLG027" H 5300 2395 50  0001 C CNN
-F 1 "PWR_FLAG" H 5300 2480 50  0000 C CNN
-F 2 "" H 5300 2300 50  0000 C CNN
-F 3 "" H 5300 2300 50  0000 C CNN
-	1    5300 2300
-	1    0    0    -1
-$EndComp
-Wire Wire Line
-	5300 2400 5300 2300
-Wire Wire Line
-	5550 2350 5300 2350
-Connection ~ 5300 2350
 $Comp
 L D_Schottky D2
@@
 $EndComp
 $Comp
-L PWR_FLAG #FLG028
+L PWR_FLAG #FLG027
 U 1 1 57747864
 P 5100 4950
-F 0 "#FLG028" H 5100 5045 50  0001 C CNN
+F 0 "#FLG027" H 5100 5045 50  0001 C CNN
 F 1 "PWR_FLAG" H 5100 5130 50  0000 C CNN
 F 2 "" H 5100 4950 50  0000 C CNN
@@
 	-1   0    0    1
 $EndComp
+$Comp
+L CONN_01X02 P10
+U 1 1 57D697B5
+P 3350 2300
+F 0 "P10" H 3350 2450 50  0000 C CNN
+F 1 "CONN_01X02" V 3450 2300 50  0000 C CNN
+F 2 "Pin_Headers:Pin_Header_Straight_1x02" H 3350 2300 50  0001 C CNN
+F 3 "" H 3350 2300 50  0000 C CNN
+	1    3350 2300
+	0    -1   -1   0
+$EndComp
+$Comp
+L GND #PWR028
+U 1 1 57D69FE6
+P 3050 2800
+F 0 "#PWR028" H 3050 2550 50  0001 C CNN
+F 1 "GND" H 3050 2650 50  0000 C CNN
+F 2 "" H 3050 2800 50  0000 C CNN
+F 3 "" H 3050 2800 50  0000 C CNN
+	1    3050 2800
+	1    0    0    -1
+$EndComp
+$Comp
+L +12V #PWR029
+U 1 1 57D6A04E
+P 3650 2650
+F 0 "#PWR029" H 3650 2500 50  0001 C CNN
+F 1 "+12V" H 3650 2790 50  0000 C CNN
+F 2 "" H 3650 2650 50  0000 C CNN
+F 3 "" H 3650 2650 50  0000 C CNN
+	1    3650 2650
+	1    0    0    -1
+$EndComp
+Wire Wire Line
+	3300 2750 3300 2500
+Wire Wire Line
+	3050 2750 3300 2750
+Wire Wire Line
+	3400 2500 3400 2750
+Wire Wire Line
+	3400 2750 3650 2750
+Wire Wire Line
+	3650 2650 3650 2800
+Connection ~ 3650 2750
+Wire Wire Line
+	5850 2300 6000 2300
+Wire Wire Line
+	6000 2300 6000 2250
+Connection ~ 5850 2300
+Wire Wire Line
+	5550 2300 5550 2100
+Text Notes 5300 1700 0    60   ~ 0
+Balancing battery\n    connector
+Wire Wire Line
+	3050 2700 3050 2800
+$Comp
+L PWR_FLAG #FLG030
+U 1 1 57D6B7F6
+P 3050 2700
+F 0 "#FLG030" H 3050 2795 50  0001 C CNN
+F 1 "PWR_FLAG" H 3050 2880 50  0000 C CNN
+F 2 "" H 3050 2700 50  0000 C CNN
+F 3 "" H 3050 2700 50  0000 C CNN
+	1    3050 2700
+	1    0    0    -1
+$EndComp
+Connection ~ 3050 2750
 $EndSCHEMATC
